File: final/final.sch (EAGLE design)
At the start: 5 parts, among them J1 POWER_JACK

Commit message: Power component
Parts:
- removed FRAME2: FRAME-LETTER, SparkFun-Aesthetics:FRAME-LETTER
- added C3, C4, C6, C7: 0.1uF, SparkFun:CAP0402-CAP
- added C5, C8: 10uf , 20V, SparkFun:CAP_POL3528
- added IC1: (no value), adafruit:MCP1700INLINE
- added JP1, JP2, JP3, JP7: (no value), SparkFun:M08LONGPADS
- added JP4: LOGO-SFESK, SparkFun:LOGO-SFESK
- added JP5, JP6: FIDUCIAL1X2, SparkFun:FIDUCIAL1X2
- added U$1: CREATIVE_COMMONS, SparkFun:CREATIVE_COMMONS
- added U1: PIC32MX250F128B-I_SP, PIC32:PIC32MX250F128B-I_SP
- added U2, U3: TB6621FNG, SparkFun:TB6621FNG
Connections:
- new net 3.3V: C2.1, IC1.OUT
- new net A01: JP1.5, JP3.5, U2.A01@1, U2.A01@2, U3.A01@1, U3.A01@2
- new net A02: JP1.4, JP3.4, U2.A02@5, U2.A02@6, U3.A02@5, U3.A02@6
- new net AIN1: JP2.3, JP7.3, U2.AIN1, U3.AIN1
- new net AIN2: JP2.2, JP7.2, U2.AIN2, U3.AIN2
- new net B01: JP1.2, JP3.2, U2.B01@11, U2.B01@12, U3.B01@11, U3.B01@12
- new net B02: JP1.3, JP3.3, U2.B02@7, U2.B02@8, U3.B02@7, U3.B02@8
- new net BIN1: JP2.5, JP7.5, U2.BIN1, U3.BIN1
- new net BIN2: JP2.6, JP7.6, U2.BIN2, U3.BIN2
- new net GND: C1.2, C2.2, C3.2, C4.2, C5.-, C6.2, C7.2, C8.-, IC1.GND, J1.GND, JP1.1, JP1.6, JP2.8, JP3.1, JP3.6, JP7.8, U2.GND, U2.PGND1@3, U2.PGND1@4, U2.PGND2@10, U2.PGND2@9, U3.GND, U3.PGND1@3, U3.PGND1@4, U3.PGND2@10, U3.PGND2@9
- new net N$1: D1.A, J1.PWR
- new net N$2: C1.1, D1.C, IC1.IN
- new net PWMA: JP2.1, JP7.1, U2.PWMA, U3.PWMA
- new net PWMB: JP2.7, JP7.7, U2.PWMB, U3.PWMB
- new net STBY: JP2.4, JP7.4, U2.STBY, U3.STBY
- new net VCC: C4.1, C7.1, JP1.7, JP3.7, U2.VCC, U3.VCC
- new net VM: C3.1, C5.+, C6.1, C8.+, JP1.8, JP3.8, U2.VM1, U2.VM2, U2.VM3, U3.VM1, U3.VM2, U3.VM3
Other:
- note added: "Peter Dokter"
- note added: "Switch"

Commit message: Update H bridge
Parts:
- removed C5, C8: 10uf , 20V, SparkFun:CAP_POL3528
- removed C6, C7: 0.1uF, SparkFun:CAP0402-CAP
- removed JP1, JP2, JP3, JP7: (no value), SparkFun:M08LONGPADS
- removed JP4: LOGO-SFESK, SparkFun:LOGO-SFESK
- removed JP5, JP6: FIDUCIAL1X2, SparkFun:FIDUCIAL1X2
- removed U$1: CREATIVE_COMMONS, SparkFun:CREATIVE_COMMONS
- removed U2, U3: TB6621FNG, SparkFun:TB6621FNG
- added IC2: L293D, st-microelectronics:L293D
- added J2, J3, J4, J5: (no value), SparkFun-Connectors:CONN_01
- C3, C4: device SparkFun:CAP0402-CAP -> SparkFun-Capacitors:0.1UF-0402-16V-10%
Connections:
- removed net A01: JP1.5, JP3.5, U2.A01@1, U2.A01@2, U3.A01@1, U3.A01@2
- removed net A02: JP1.4, JP3.4, U2.A02@5, U2.A02@6, U3.A02@5, U3.A02@6
- removed net AIN1: JP2.3, JP7.3, U2.AIN1, U3.AIN1
- removed net AIN2: JP2.2, JP7.2, U2.AIN2, U3.AIN2
- removed net B01: JP1.2, JP3.2, U2.B01@11, U2.B01@12, U3.B01@11, U3.B01@12
- removed net B02: JP1.3, JP3.3, U2.B02@7, U2.B02@8, U3.B02@7, U3.B02@8
- removed net BIN1: JP2.5, JP7.5, U2.BIN1, U3.BIN1
- removed net BIN2: JP2.6, JP7.6, U2.BIN2, U3.BIN2
- removed net PWMA: JP2.1, JP7.1, U2.PWMA, U3.PWMA
- removed net PWMB: JP2.7, JP7.7, U2.PWMB, U3.PWMB
- removed net STBY: JP2.4, JP7.4, U2.STBY, U3.STBY
- removed net VCC: C4.1, C7.1, JP1.7, JP3.7, U2.VCC, U3.VCC
- removed net VM: C3.1, C5.+, C6.1, C8.+, JP1.8, JP3.8, U2.VM1, U2.VM2, U2.VM3, U3.VM1, U3.VM2, U3.VM3
- new net 12V: C3.1, IC2.VCC1, IC2.VCC2
- new net MC1_1: IC2.1A, U1.OSC1/CLKI/RPA2/RA2
- new net MC1_2: IC2.2A, U1.OSC2/CLKO/RPA3/PMA0/RA3
- new net MC2_1: IC2.4A, U1.PGEC2/RPB11/D-/RB11
- new net MC2_2: IC2.3A, U1.PGED2/RPB10/D+/CTED11/RB10
- net 3.3V: now also IC2.1-2EN, IC2.3-4EN
- net GND: now also IC2.GND1, IC2.GND2, IC2.GND3, IC2.GND4, J1.GNDBREAK; no longer C4.2, C5.-, C6.2, C7.2, C8.-, JP1.1, JP1.6, JP2.8, JP3.1, JP3.6, JP7.8, U2.GND, U2.PGND1@3, U2.PGND1@4, U2.PGND2@10, U2.PGND2@9, U3.GND, U3.PGND1@3, U3.PGND1@4, U3.PGND2@10, U3.PGND2@9
Other:
- note removed: "Peter Dokter"
